File: Boards/Controller1/Controller1.brd (EAGLE design)
At the start: 81.3 x 77.1 mm, 9 parts

Commit message: removed obsolete signals
Connections:
- removed net BLE_CS: MCU1.16
- removed net BLE_IRQ: MCU1.15
- removed net BLE_MISO: MCU1.19
- removed net BLE_MOSI: MCU1.17
- removed net BLE_SCK: MCU1.18
Changed lines of the file:
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@@
 </elements>
 <signals>
-<signal name="BLE_SCK">
-<contactref element="MCU1" pad="18"/>
-</signal>
-<signal name="BLE_MISO">
-<contactref element="MCU1" pad="19"/>
-</signal>
-<signal name="BLE_MOSI">
-<contactref element="MCU1" pad="17"/>
-</signal>
-<signal name="BLE_CS">
-<contactref element="MCU1" pad="16"/>
-</signal>
 <signal name="GND">
 <contactref element="MCU1" pad="25"/>
@@
 <wire x1="44.5" y1="66" x2="44.45" y2="66.04" width="1.27" layer="1"/>
 </signal>
-<signal name="BLE_IRQ">
-<contactref element="MCU1" pad="15"/>
-</signal>
 <signal name="12V">
