File: Boards/PositionSensor/PositionSensor.sch (EAGLE design)
At the start: 4 parts

Commit message: finished for mass production
Connections:
- net VCC renamed 3V3
Changed lines of the file:
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@@
-</segment>
-</net>
-<net name="VCC" class="0">
-<segment>
-<pinref part="R1" gate="G$1" pin="2"/>
-<wire x1="35.56" y1="55.88" x2="5.08" y2="55.88" width="0.1524" layer="91"/>
-<pinref part="R2" gate="G$1" pin="1"/>
-<label x="17.78" y="55.88" size="1.778" layer="95"/>
-</segment>
-<segment>
-<pinref part="J1" gate="J$1" pin="1"/>
-<wire x1="17.78" y1="7.62" x2="30.48" y2="7.62" width="0.1524" layer="91"/>
-<label x="20.32" y="7.62" size="1.778" layer="95"/>
 </segment>
 </net>
@@
 </segment>
 </net>
+<net name="3V3" class="0">
+<segment>
+<pinref part="J1" gate="J$1" pin="1"/>
+<wire x1="17.78" y1="7.62" x2="30.48" y2="7.62" width="0.1524" layer="91"/>
+<label x="20.32" y="7.62" size="1.778" layer="95"/>
+</segment>
+<segment>
+<pinref part="R1" gate="G$1" pin="2"/>
+<wire x1="35.56" y1="55.88" x2="5.08" y2="55.88" width="0.1524" layer="91"/>
+<pinref part="R2" gate="G$1" pin="1"/>
+<label x="17.78" y="55.88" size="1.778" layer="95"/>
+</segment>
+</net>
